File: hardware/PCBot.kicad_sch (KiCad schematic)
At the start: 61 parts, among them J101 Conn_ST_STDC14, M101 Motor_DC_ALT, M102 Motor_DC_ALT, U101 STM32G431CBUx, U102 AMS1117-3.3, U103 LSM6DS3, U104 STSPIN250, U105 STSPIN250, Y101 Crystal_GND24_DNP

Commit message: initial commit 420
Signed-off-by: Connor Rigby <connorr@hey.com>
Parts:
- added H101, H102, H103, H104, H105, H106, H107, H108: MountingHole_Pad, LCSC_Connector:SMD_BD5.6-L5.6-W5.6-D3.6, symbol Mechanical:MountingHole_Pad
- added SW101: SW_SPDT, LCSC_Switch:SW-TH_SS-12D16L3R, symbol Switch:SW_SPDT
- BT101, M101: footprint LCSC_Connector:PAD_01x02 -> (none); now left out of the parts list
- M102: now left out of the parts list
Connections:
- net +BATT: now also SW101.3 (C); no longer BT101.1 (+)
- net GND: now also H101.1, H102.1, H103.1, H104.1, H105.1, H106.1, H107.1, H108.1
- new net: BT101.1 (+), SW101.2 (B)
- no-connect marks 2 -> 3
Other:
- moved on the sheet: BT101, C107, C108, U102

Commit message: initial commit
Signed-off-by: Connor Rigby <connorr@hey.com>
Parts:
- removed C104, C111: C_0402_1nf_X7R, Capacitor_SMD:C_0402_1005Metric, symbol LCSC_Capacitor:C_0402_1nf_X7R
- removed D102, D103: GREEN, LED_SMD:LED_0402_1005Metric, symbol Device:LED_Small
- removed D104, D105: RED, LED_SMD:LED_0402_1005Metric, symbol Device:LED_Small
- removed R114, R115: R_0402_4k7, Resistor_SMD:R_0402_1005Metric, symbol LCSC_Resistor:R_0402_4k7
- removed R116: R_0402_1k, Resistor_SMD:R_0402_1005Metric, symbol LCSC_Resistor:R_0402_1k
- removed RN102: RA_0402_04_DNP, Resistor_SMD:R_Array_Concave_4x0402, symbol LCSC_Resistor:RA_0402_04_DNP
- added BT102: Battery_Cell, Battery:BatteryHolder_Seiko_MS621F, symbol Device:Battery_Cell
- added C104, C111: C_0402_DNP, Capacitor_SMD:C_0402_1005Metric, symbol LCSC_Capacitor:C_0402_DNP
- added C129, C130: C_0805_4u7_X5R, Capacitor_SMD:C_0805_2012Metric, symbol LCSC_Capacitor:C_0805_4u7_X5R
- added C131, C132: C_0805_1u_X7R, Capacitor_SMD:C_0805_2012Metric, symbol LCSC_Capacitor:C_0805_1u_X7R
- added D106: BAT54C, Package_TO_SOT_SMD:SOT-23, symbol Diode:BAT54C
- added JM1: JM1, Connector_PinHeader_2.00mm:PinHeader_1x06_P2.00mm_Horizontal, symbol Connector_Generic:Conn_01x06
- added JM2: JM2, Connector_PinHeader_2.00mm:PinHeader_1x06_P2.00mm_Horizontal, symbol Connector_Generic:Conn_01x06
- added R114: R_0402_1k, Resistor_SMD:R_0402_1005Metric, symbol LCSC_Resistor:R_0402_1k
- added R115, R116: R_1206_DNP, Resistor_SMD:R_1206_3216Metric, symbol LCSC_Resistor:R_1206_DNP
- added TP101: RESET, TestPoint:TestPoint_Pad_D1.0mm, symbol Connector:TestPoint
- added TP102: VDD, TestPoint:TestPoint_Pad_4.0x4.0mm, symbol Connector:TestPoint
- added TP103: GND, TestPoint:TestPoint_Pad_4.0x4.0mm, symbol Connector:TestPoint
- added Y102: Q13FC1350000400, Crystal:Crystal_SMD_3215-2Pin_3.2x1.5mm, symbol LCSC_Crystal:Q13FC1350000400
- C124: now not fitted; now left out of the parts list
- R102, R107: value 18k -> 39k
Connections:
- net RF_IRQ is gone; now on net IMU_NSS: U101.16 (PC4)
- net SPI1_MOSI is gone; now on net M1_SENSE: U101.15 (PA7)
- net SPI1_SCK is gone; now on net M1_PWM: U101.13 (PA5)
- net GND: now also BT102.2 (-), C104.2, C111.2, C129.2, C130.2, C131.2, C132.2, JM1.6 (Pin_6), JM2.6 (Pin_6), R115.2, R116.2, TP103.1
- net LPUART1_RX: now also U101.22 (PB10); no longer U101.11 (PA3)
- net LPUART1_TX: now also U101.24 (PB11); no longer U101.10 (PA2)
- net M1_EN_FAULT: now also R102.1, U101.44 (PB6); no longer R102.2, U101.29 (PC6)
- net M1_OUTA1: now also JM1.2 (Pin_2)
- net M1_OUTA2: now also JM1.1 (Pin_1)
- net M1_PWM: no longer U101.30 (PA8)
- net M1_SENSE: now also R115.1; no longer U101.26 (PB13)
- net M2_EN_FAULT: now also R107.1, U101.45 (PB7); no longer R107.2, U101.28 (PB15)
- net M2_OUTA1: now also JM2.1 (Pin_1)
- net M2_OUTA2: now also JM2.2 (Pin_2)
- net M2_PWM: now also U101.9 (PA1); no longer U101.31 (PA9)
- net M2_SENSE: now also U101.17 (PB0), R116.1; no longer U101.27 (PB14)
- net VBATT_SENSE: now also U101.18 (PB1); no longer U101.8 (PA0)
- net VDD: now also R102.2, R107.2, C130.1, C131.1, C132.1, D106.2, JM1.3 (Pin_3), JM2.3 (Pin_3), R114.1, TP102.1; no longer C115.1, U101.1 (VBAT)
- net VDDA: no longer U104.11 (REF), U105.11 (REF)
- net VBAT_IN: now reaches BT101.1 (+), SW101.2 (B)
- net IMU_IRQ1: now reaches U101.2 (PC13)
- net IMU_IRQ1: now also U103.4 (INT1)
- net OSC32_IN: now reaches U101.3 (PC14)
- net OSC32_IN: now also C104.1, Y102.1
- net SPI3_SCK: now reaches U101.39 (PC10)
- net SPI3_SCK: now also U103.13 (SCL)
- net OSC32_OUT: now reaches U101.4 (PC15)
- net OSC32_OUT: now also C111.1, Y102.2
- net SPI3_MISO: now reaches U101.40 (PC11)
- net SPI3_MISO: now also U103.1 (SDO/SA0)
- net JTRST: now reaches U101.42 (PB4)
- net JTRST: now also J101.12 (~{RST})
- net I2C1_SCL renamed M2_ENC_N
- net M2_ENC_N: now also JM2.5 (Pin_5); no longer U103.13 (SCL)
- net I2C1_SDA renamed SPI3_MOSI
- net SPI3_MOSI: now also U101.43 (PB5); no longer U101.45 (PB7)
- net IMU_CS renamed IMU_NSS
- net IMU_I2C_CONFIG: no longer names the net of R113.2, U103.2 (SDX)
- net IMU_I2C_CONFIG: no longer U103.1 (SDO/SA0), U103.3 (SCX)
- removed net IMU_INT1: U101.43 (PB5), U103.4 (INT1)
- net IMU_INT2 renamed IMU_IRQ2
- net IMU_IRQ2: now also U101.10 (PA2); no longer U101.44 (PB6)
- net M1_EN renamed M1_DIR
- net M1_DIR: now also U104.1 (PH); no longer R102.1
- net M1_PH renamed VBAT_STATUS
- net VBAT_STATUS: no longer U104.1 (PH)
- removed net M2_EN: R107.1, U101.24 (PB11)
- net M2_PH renamed M2_DIR
- net MC_STBY_RESET renamed ~{RESET}
- net ~{RESET}: now also C124.1, U101.7 (PG10), TP101.1; no longer U101.25 (PB12)
- net SPI1_MISO renamed M1_REF
- net M1_REF: now also U104.11 (REF)
- net SYS_JTCK renamed JTCK
- net SYS_JTDI renamed JTDI
- net SYS_JTDO renamed JTDO
- net SYS_JTMS renamed JTMS
- removed net ~{RST}: C124.1, J101.12 (~{RST}), U101.7 (PG10)
- net ~{SPI1_SS} renamed M2_REF
- net M2_REF: now also U105.11 (REF)
- new net: C115.1, C129.1, D106.3, U101.1 (VBAT)
- new net: R114.2, U103.3 (SCX)
- new net M1_ENC_N: JM1.5 (Pin_5), U101.31 (PA9)
- new net M1_ENC_P: JM1.4 (Pin_4), U101.30 (PA8)
- new net M2_ENC_P: JM2.4 (Pin_4), U101.29 (PC6)
- new net OPAMP1_WINP: U101.11 (PA3)
- new net RADIO_IRQ: U101.8 (PA0)
- new net RADIO_NSS: U101.25 (PB12)
- new net SPI2_MISO: U101.27 (PB14)
- new net SPI2_MOSI: U101.28 (PB15)
- new net SPI2_SCK: U101.26 (PB13)
- new net VBACKUP: BT102.1 (+), D106.1
- no-connect marks 3 -> 2
Other:
- note removed: "STATUS LEDS"
- moved on the sheet: C102, C115, C116, C117, C118, C119, C120, C121, FB101, M101, M102, R102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
