File: hardware/RF_Transciever.kicad_sch (KiCad schematic)
At the start: 29 parts, among them U103 A7105, Y201 Crystal_GND24_DNP

Commit message: initial commit
Signed-off-by: Connor Rigby <connorr@hey.com>
Parts:
- removed C201: C_0402_2u2_X5R, Capacitor_SMD:C_0402_1005Metric, symbol LCSC_Capacitor:C_0402_2u2_X5R
- added C201: C_805_DNP, Capacitor_SMD:C_0805_2012Metric, symbol LCSC_Capacitor:C_805_DNP
- AE201: footprint RF_Antenna:Texas_SWRA117D_2.4GHz_Left -> (none)
Connections:
- net GND: now also C201.2
- net REG0A: now also C201.1
Changed lines of the file:
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@@
-    )
-  )
-  (symbol (lib_id "LCSC_Capacitor:C_0402_2u2_X5R") (at 139.7 53.34 0) (unit 1)
-    (in_bom yes) (on_board yes) (dnp no) (fields_autoplaced)
-    (property "Reference" "C201" (at 142.24 52.7113 0)
-      (effects (font (size 1.27 1.27)) (justify left))
-    )
-    (property "Value" "C_0402_2u2_X5R" (at 139.954 55.372 0)
-      (effects (font (size 1.27 1.27)) (justify left) hide)
-    )
-    (property "Footprint" "Capacitor_SMD:C_0402_1005Metric" (at 139.7 53.34 0)
-      (effects (font (size 1.27 1.27)) hide)
-    )
-    (property "Datasheet" "https://datasheet.lcsc.com/lcsc/1912111437_Murata-Electronics-GRM155R61E225KE11D_C385032.pdf" (at 139.7 53.34 0)
-      (effects (font (size 1.27 1.27)) hide)
-    )
-    (property "Capacitance" "2.2uF" (at 142.24 55.2513 0)
-      (effects (font (size 1.27 1.27)) (justify left))
-    )
-    (property "LCSC" "C385032" (at 139.7 53.34 0)
-      (effects (font (size 1.27 1.27)) hide)
-    )
-    (property "MPN" "GRM155R61E225KE11D" (at 139.7 53.34 0)
-      (effects (font (size 1.27 1.27)) hide)
-    )
-    (property "Voltage" "25V" (at 139.7 53.34 0)
-      (effects (font (size 1.27 1.27)) hide)
-    )
-    (property "Tolerance" "10%" (at 139.7 53.34 0)
-      (effects (font (size 1.27 1.27)) hide)
-    )
-    (property "Temperature" "X5R" (at 139.7 53.34 0)
-      (effects (font (size 1.27 1.27)) hide)
-    )
-    (pin "1")
-    (pin "2")
-    (instances
-      (project "PCBot"
-        (path "/46741512-c7c8-4a4b-b9b2-a5eb78354a7c/408f8330-5e10-4a1d-89b1-14802b0f9bea"
-          (reference "C201") (unit 1)
-        )
-      )
     )
   )
@@
     )
   )
+  (symbol (lib_id "LCSC_Capacitor:C_805_DNP") (at 139.7 53.34 0) (unit 1)
+    (in_bom no) (on_board yes) (dnp no) (fields_autoplaced)
+    (property "Reference" "C201" (at 142.24 52.7113 0)
+      (effects (font (size 1.27 1.27)) (justify left))
+    )
+    (property "Value" "C_805_DNP" (at 139.954 55.372 0)
+      (effects (font (size 1.27 1.27)) (justify left) hide)
+    )
+    (property "Footprint" "Capacitor_SMD:C_0805_2012Metric" (at 139.7 53.34 0)
+      (effects (font (size 1.27 1.27)) hide)
+    )
+    (property "Datasheet" "~" (at 139.7 53.34 0)
+      (effects (font (size 1.27 1.27)) hide)
+    )
+    (property "Capacitance" "DNP" (at 142.24 55.2513 0)
+      (effects (font (size 1.27 1.27)) (justify left))
+    )
+    (pin "1")
+    (pin "2")
+    (instances
+      (project "PCBot"
+        (path "/46741512-c7c8-4a4b-b9b2-a5eb78354a7c/408f8330-5e10-4a1d-89b1-14802b0f9bea"
+          (reference "C201") (unit 1)
+        )
+      )
+    )
+  )
   (symbol (lib_id "power:GND") (at 157.48 104.14 0) (unit 1)
     (in_bom yes) (on_board yes) (dnp no) (fields_autoplaced)
@@
       (effects (font (size 1.27 1.27)) (justify right))
     )
-    (property "Footprint" "RF_Antenna:Texas_SWRA117D_2.4GHz_Left" (at 38.1 43.815 0)
-      (effects (font (size 1.27 1.27)) hide)
-    )
+    (property "Footprint" "" (at 38.1 43.815 0)
+      (effects (font (size 1.27 1.27)) hide)
+    )
