File: hardware/PCBot.kicad_pcb (KiCad board)
At the start: 4 copper layers, 68 x 37 mm, 101 parts, among them J101 Conn_ST_STDC14, M101 Motor_DC_ALT, M102 Motor_DC_ALT, U101 STM32G431CBUx, U102 AMS1117-3.3, U103 LSM6DS3, U104 STSPIN250, U105 STSPIN250, U201 A7105, Y101 Crystal_GND24_DNP, Y201 Crystal_GND24_DNP

Commit message: initial commit 3
Signed-off-by: Connor Rigby <connorr@hey.com>
Parts:
- removed AE201: Antenna_Chip, RF_Antenna:Texas_SWRA117D_2.4GHz_Left
- removed BT101: Battery, LCSC_Connector:PAD_01x02
- removed C101, C102, C103, C109, C110, C114, C127, C128, C203, C206, C207, C208, C209, C211, C214, C215, C216, C217, C218, C219, C220: C_0402_DNP, Capacitor_SMD:C_0402_1005Metric
- removed C104, C111: C_0402_1nf_X7R, Capacitor_SMD:C_0402_1005Metric
- removed C105, C112: C_805_DNP, Capacitor_SMD:C_0805_2012Metric
- removed C106, C113: 22uf, Capacitor_SMD:CP_Elec_4x5.4
- removed C107: C_0805_1u_X7R, Capacitor_SMD:C_0805_2012Metric
- removed C108: C_0805_10u_X5R, Capacitor_SMD:C_0805_2012Metric
- removed C115, C116, C117, C118, C119, C122, C123, C124, C125, C126, C205: C_0402_100nf_X7R, Capacitor_SMD:C_0402_1005Metric
- removed C120: C_0805_4u7_X5R, Capacitor_SMD:C_0805_2012Metric
- removed C121: C_0402_1u_X5R, Capacitor_SMD:C_0402_1005Metric
- removed C201, C202, C204: C_0402_2u2_X5R, Capacitor_SMD:C_0402_1005Metric
- removed C210: C_0402_22p_C0G, Capacitor_SMD:C_0402_1005Metric
- removed C212: C_0402_100p_C0G, Capacitor_SMD:C_0402_1005Metric
- removed C213: C_0402_10n_C0G, Capacitor_SMD:C_0402_1005Metric
- removed D101: 30v 230mv@100ma 1A, Diode_SMD:D_SOD-323F
- removed FB101: FerriteBead_Small, Inductor_SMD:L_0402_1005Metric
- removed J101: Conn_ST_STDC14, LCSC_Connector:TC2070-IDC-FP
- removed L202, L203, L204: L_0402_DNP, Inductor_SMD:L_0402_1005Metric
- removed M101, M102: Motor_DC_ALT, LCSC_Connector:PAD_01x02
- removed R101, R102, R103, R106, R107, R110: 18k, Resistor_SMD:R_0402_1005Metric
- removed R104, R109, R113, R116: R_0402_1k, Resistor_SMD:R_0402_1005Metric
- removed R105, R108: R_1206_DNP, Resistor_SMD:R_1206_3216Metric
- removed R111, R112: R_0603_DNP, Resistor_SMD:R_0603_1608Metric
- removed R114, R115: R_0402_4k7, Resistor_SMD:R_0402_1005Metric
- removed R201, R203: DNP, Resistor_SMD:R_0402_1005Metric
- removed R202: 200, Resistor_SMD:R_0402_1005Metric
- removed REF** (x5): MountingHole_2.2mm_M2_Pad_Via, MountingHole:MountingHole_2.2mm_M2_Pad_Via
- removed U101: STM32G431CBUx, Package_DFN_QFN:QFN-48-1EP_7x7mm_P0.5mm_EP5.6x5.6mm
- removed U102: AMS1117-3.3, Package_TO_SOT_SMD:SOT-223-3_TabPin2
- removed U103: LSM6DS3, Package_LGA:LGA-14_3x2.5mm_P0.5mm_LayoutBorder3x4y
- removed U104, U105: STSPIN250, Package_DFN_QFN:TQFN-16-1EP_3x3mm_P0.5mm_EP1.6x1.6mm
- removed U201: A7105, Package_DFN_QFN:QFN-20-1EP_4x4mm_P0.5mm_EP2.5x2.5mm
- removed Y101, Y201: Crystal_GND24_DNP, Crystal:Crystal_SMD_3225-4Pin_3.2x2.5mm
- removed kibuzzard-646A62D2: G***, kibuzzard-646A62D2
- removed kibuzzard-646A6321: G***, kibuzzard-646A6321
- removed kibuzzard-646A63AE (x2): G***, kibuzzard-646A63AE
- removed kibuzzard-646A6533 (x2): G***, kibuzzard-646A6533
- removed kibuzzard-646A657B (x2): G***, kibuzzard-646A657B
- removed kibuzzard-646A6855: G***, kibuzzard-646A6855
- removed kibuzzard-646A6AA4: G***, kibuzzard-646A6AA4
- removed kibuzzard-646A6DD1: G***, kibuzzard-646A6DD1
Routing:
- net GND: track 90.8 -> 0.00 mm, vias 95 -> 0
- net /SYS_JTDI: track 72.9 -> 0.00 mm, vias 2 -> 0
- net /M2_SENSE: track 70.6 -> 0.00 mm, vias 4 -> 0
- net VDDA: track 67.8 -> 0.00 mm, vias 3 -> 0
- net /M1_SENSE: track 66.1 -> 0.00 mm, vias 4 -> 0
- net /MC_STBY_RESET: track 60.4 -> 0.00 mm, vias 4 -> 0
- net /SYS_JTDO: track 56.8 -> 0.00 mm, vias 2 -> 0
- net /M2_EN: track 51.9 -> 0.00 mm, vias 2 -> 0
- net /M2_EN_FAULT: track 50.7 -> 0.00 mm
- net VDD: track 48.6 -> 0.00 mm, vias 20 -> 0
- net /SYS_JTCK: track 48.2 -> 0.00 mm, vias 2 -> 0
- net /SYS_JTMS: track 45.8 -> 0.00 mm, vias 2 -> 0
- net /M2_PWM: track 43.6 -> 0.00 mm, vias 2 -> 0
- net /VBATT_SENSE: track 42.9 -> 0.00 mm, vias 2 -> 0
- net /M1_EN_FAULT: track 41.8 -> 0.00 mm, vias 2 -> 0
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- removed copper zone on F.Cu, net +BATT
- removed copper zone on B.Cu, net /M1_OUTA1
- removed copper zone on F.Cu, net /M1_OUTA1
- removed copper zone on B.Cu, net /M1_OUTA2
- removed copper zone on F.Cu, net /M1_OUTA2
- removed copper zone on B.Cu, net /M2_OUTA1
- removed copper zone on F.Cu, net /M2_OUTA1
- removed copper zone on B.Cu, net /M2_OUTA2
- removed copper zone on F.Cu, net /M2_OUTA2
- removed copper zone on B.Cu, net GND
- removed copper zone on F.Cu, net GND
- removed copper zone on F.Cu, net VDD
Other:
- board size 68 x 37 mm -> 70 x 60 mm
- board text removed: "Rev.1"
- board text removed: "X"
- board text removed: "Y"
- board text removed: "Z"

Commit message: uhhhhhhhhhhhhhhhhhhhhhhhh
Signed-off-by: Connor Rigby <connorr@hey.com>
Parts:
- added REF**: SMD_BD5.6-L5.6-W5.6-D3.6, LCSC_Connector:SMD_BD5.6-L5.6-W5.6-D3.6, F.Cu at (116.8, 22.9)
- added REF**: SMD_BD5.6-L5.6-W5.6-D3.6, LCSC_Connector:SMD_BD5.6-L5.6-W5.6-D3.6, F.Cu at (84.5, 67.2)
- added REF**: SMD_BD5.6-L5.6-W5.6-D3.6, LCSC_Connector:SMD_BD5.6-L5.6-W5.6-D3.6, F.Cu at (23.8, 69.0)
- added REF**: SMD_BD5.6-L5.6-W5.6-D3.6, LCSC_Connector:SMD_BD5.6-L5.6-W5.6-D3.6, F.Cu at (56.0, 33.6)
- added REF**: SMD_BD5.6-L5.6-W5.6-D3.6, LCSC_Connector:SMD_BD5.6-L5.6-W5.6-D3.6, F.Cu at (56.0, 67.3)
- added REF**: SMD_BD5.6-L5.6-W5.6-D3.6, LCSC_Connector:SMD_BD5.6-L5.6-W5.6-D3.6, F.Cu at (33.8, 81.9)
- added REF**: SMD_BD5.6-L5.6-W5.6-D3.6, LCSC_Connector:SMD_BD5.6-L5.6-W5.6-D3.6, F.Cu at (84.6, 33.6)
- added REF**: SMD_BD5.6-L5.6-W5.6-D3.6, LCSC_Connector:SMD_BD5.6-L5.6-W5.6-D3.6, F.Cu at (116.8, 68.9)
- added REF**: SMD_BD5.6-L5.6-W5.6-D3.6, LCSC_Connector:SMD_BD5.6-L5.6-W5.6-D3.6, F.Cu at (23.8, 23.0)
- added REF**: SMD_BD5.6-L5.6-W5.6-D3.6, LCSC_Connector:SMD_BD5.6-L5.6-W5.6-D3.6, F.Cu at (106.8, 81.9)
Other:
- board size 70 x 60 mm -> 100 x 65 mm

Commit message: initial commit 69
Signed-off-by: Connor Rigby <connorr@hey.com>
Parts:
- removed the REF** at (116.8, 22.9)
- removed the REF** at (84.5, 67.2)
- removed the REF** at (23.8, 69.0)
- removed the REF** at (56.0, 33.6)
- removed the REF** at (56.0, 67.3)
- removed the REF** at (33.8, 81.9)
- removed the REF** at (84.6, 33.6)
- removed the REF** at (116.8, 68.9)
- removed the REF** at (23.8, 23.0)
- removed the REF** at (106.8, 81.9)
- added BT101: Battery, LCSC_Connector:PAD_01x02, F.Cu at (68.6, 36.0)
- added C101: C_0402_DNP, Capacitor_SMD:C_0402_1005Metric, F.Cu at (105.1, 43.2)
- added C102: C_0402_DNP, Capacitor_SMD:C_0402_1005Metric, F.Cu at (105.1, 45.1)
- added C103: C_0402_DNP, Capacitor_SMD:C_0402_1005Metric, F.Cu at (105.1, 47.1)
- added C104: C_0402_1nf_X7R, Capacitor_SMD:C_0402_1005Metric, F.Cu at (105.1, 49.1)
- added C105: C_805_DNP, Capacitor_SMD:C_0805_2012Metric, F.Cu at (112.2, 47.0)
- added C106: 22uf, Capacitor_SMD:CP_Elec_4x5.4, F.Cu at (104.6, 39.2)
- added C107: C_0805_1u_X7R, Capacitor_SMD:C_0805_2012Metric, F.Cu at (68.9, 44.0)
- added C108: C_0805_10u_X5R, Capacitor_SMD:C_0805_2012Metric, F.Cu at (71.9, 44.0)
- added C109: C_0402_DNP, Capacitor_SMD:C_0402_1005Metric, F.Cu at (48.1, 43.0)
- added C110: C_0402_DNP, Capacitor_SMD:C_0402_1005Metric, F.Cu at (48.1, 44.9)
- added C111: C_0402_1nf_X7R, Capacitor_SMD:C_0402_1005Metric, F.Cu at (48.1, 46.9)
- added C112: C_805_DNP, Capacitor_SMD:C_0805_2012Metric, F.Cu at (55.2, 46.8)
- added C113: 22uf, Capacitor_SMD:CP_Elec_4x5.4, F.Cu at (47.6, 39.0)
- added C114: C_0402_DNP, Capacitor_SMD:C_0402_1005Metric, F.Cu at (48.1, 48.9)
- added C115: C_0402_100nf_X7R, Capacitor_SMD:C_0402_1005Metric, F.Cu at (101.3, 88.2)
- added C116: C_0402_100nf_X7R, Capacitor_SMD:C_0402_1005Metric, F.Cu at (101.3, 90.1)
- added C117: C_0402_100nf_X7R, Capacitor_SMD:C_0402_1005Metric, F.Cu at (101.3, 92.1)
- added C118: C_0402_100nf_X7R, Capacitor_SMD:C_0402_1005Metric, F.Cu at (104.1, 88.2)
- added C119: C_0402_100nf_X7R, Capacitor_SMD:C_0402_1005Metric, F.Cu at (104.1, 90.1)
- added C120: C_0805_4u7_X5R, Capacitor_SMD:C_0805_2012Metric, F.Cu at (111.3, 79.4)
- added C121: C_0402_1u_X5R, Capacitor_SMD:C_0402_1005Metric, F.Cu at (104.1, 92.1)
- added C122: C_0402_100nf_X7R, Capacitor_SMD:C_0402_1005Metric, F.Cu at (107.0, 88.2)
- added C123: C_0402_100nf_X7R, Capacitor_SMD:C_0402_1005Metric, F.Cu at (50.4, 83.9)
- added C124: C_0402_100nf_X7R, Capacitor_SMD:C_0402_1005Metric, F.Cu at (50.4, 85.9)
- added C125: C_0402_100nf_X7R, Capacitor_SMD:C_0402_1005Metric, F.Cu at (50.4, 95.5)
- added C126: C_0402_100nf_X7R, Capacitor_SMD:C_0402_1005Metric, F.Cu at (50.4, 97.5)
- added C127: C_0402_DNP, Capacitor_SMD:C_0402_1005Metric, F.Cu at (107.0, 90.1)
- added C128: C_0402_DNP, Capacitor_SMD:C_0402_1005Metric, F.Cu at (107.0, 92.1)
- added C201: C_0402_2u2_X5R, Capacitor_SMD:C_0402_1005Metric, F.Cu at (74.1, 91.7)
- added C202: C_0402_2u2_X5R, Capacitor_SMD:C_0402_1005Metric, F.Cu at (74.1, 93.7)
- added C203: C_0402_DNP, Capacitor_SMD:C_0402_1005Metric, F.Cu at (74.1, 95.6)
- added C204: C_0402_2u2_X5R, Capacitor_SMD:C_0402_1005Metric, F.Cu at (74.1, 97.6)
- added C205: C_0402_100nf_X7R, Capacitor_SMD:C_0402_1005Metric, F.Cu at (74.1, 99.6)
- added C206: C_0402_DNP, Capacitor_SMD:C_0402_1005Metric, F.Cu at (77.0, 91.7)
- added C207: C_0402_DNP, Capacitor_SMD:C_0402_1005Metric, F.Cu at (77.0, 93.7)
- added C208: C_0402_DNP, Capacitor_SMD:C_0402_1005Metric, F.Cu at (77.0, 95.6)
- added C209: C_0402_DNP, Capacitor_SMD:C_0402_1005Metric, F.Cu at (77.0, 97.6)
- added C210: C_0402_22p_C0G, Capacitor_SMD:C_0402_1005Metric, F.Cu at (77.0, 99.6)
- added C211: C_0402_DNP, Capacitor_SMD:C_0402_1005Metric, F.Cu at (79.9, 91.7)
- added C212: C_0402_100p_C0G, Capacitor_SMD:C_0402_1005Metric, F.Cu at (79.9, 93.7)
- added C213: C_0402_10n_C0G, Capacitor_SMD:C_0402_1005Metric, F.Cu at (79.9, 95.6)
- added C214: C_0402_DNP, Capacitor_SMD:C_0402_1005Metric, F.Cu at (79.9, 97.6)
- added C215: C_0402_DNP, Capacitor_SMD:C_0402_1005Metric, F.Cu at (79.9, 99.6)
- added C216: C_0402_DNP, Capacitor_SMD:C_0402_1005Metric, F.Cu at (82.7, 91.7)
- added C217: C_0402_DNP, Capacitor_SMD:C_0402_1005Metric, F.Cu at (82.7, 93.7)
- added C218: C_0402_DNP, Capacitor_SMD:C_0402_1005Metric, F.Cu at (82.7, 95.6)
- added C219: C_0402_DNP, Capacitor_SMD:C_0402_1005Metric, F.Cu at (82.7, 97.6)
- added C220: C_0402_DNP, Capacitor_SMD:C_0402_1005Metric, F.Cu at (82.7, 99.6)
- added D101: 30v 230mv@100ma 1A, Diode_SMD:D_SOD-323F, F.Cu at (46.8, 84.4)
- added FB101: FerriteBead_Small, Inductor_SMD:L_0402_1005Metric, F.Cu at (110.6, 81.9)
- added J101: Conn_ST_STDC14, LCSC_Connector:TC2070-IDC-FP, F.Cu at (58.8, 75.9)
- added L202: L_0402_DNP, Inductor_SMD:L_0402_1005Metric, F.Cu at (71.2, 91.7)
- added L203: L_0402_DNP, Inductor_SMD:L_0402_1005Metric, F.Cu at (71.2, 93.7)
- added L204: L_0402_DNP, Inductor_SMD:L_0402_1005Metric, F.Cu at (71.2, 95.7)
- added M101: Motor_DC_ALT, LCSC_Connector:PAD_01x02, F.Cu at (108.3, 46.7)
- added M102: Motor_DC_ALT, LCSC_Connector:PAD_01x02, F.Cu at (51.3, 46.5)
- added R101: 18k, Resistor_SMD:R_0402_1005Metric, F.Cu at (102.2, 43.2)
- added R102: 18k, Resistor_SMD:R_0402_1005Metric, F.Cu at (102.2, 45.2)
- added R103: 18k, Resistor_SMD:R_0402_1005Metric, F.Cu at (102.2, 47.1)
- added R104: R_0402_1k, Resistor_SMD:R_0402_1005Metric, F.Cu at (102.2, 49.1)
- added R105: R_1206_DNP, Resistor_SMD:R_1206_3216Metric, F.Cu at (109.3, 43.8)
- added R106: 18k, Resistor_SMD:R_0402_1005Metric, F.Cu at (45.2, 43.0)
- added R107: 18k, Resistor_SMD:R_0402_1005Metric, F.Cu at (45.2, 45.0)
- added R108: R_1206_DNP, Resistor_SMD:R_1206_3216Metric, F.Cu at (52.3, 43.6)
- added R109: R_0402_1k, Resistor_SMD:R_0402_1005Metric, F.Cu at (45.2, 47.0)
- added R110: 18k, Resistor_SMD:R_0402_1005Metric, F.Cu at (45.2, 48.9)
- added R111: R_0603_DNP, Resistor_SMD:R_0603_1608Metric, F.Cu at (68.6, 39.8)
- added R112: R_0603_DNP, Resistor_SMD:R_0603_1608Metric, F.Cu at (71.2, 39.8)
- added R113: R_0402_1k, Resistor_SMD:R_0402_1005Metric, F.Cu at (47.5, 91.5)
- added R114: R_0402_4k7, Resistor_SMD:R_0402_1005Metric, F.Cu at (47.5, 93.5)
- added R115: R_0402_4k7, Resistor_SMD:R_0402_1005Metric, F.Cu at (47.5, 95.5)
- added R116: R_0402_1k, Resistor_SMD:R_0402_1005Metric, F.Cu at (47.5, 97.5)
- added R201: DNP, Resistor_SMD:R_0402_1005Metric, F.Cu at (71.2, 97.7)
- added R202: 200, Resistor_SMD:R_0402_1005Metric, F.Cu at (71.2, 99.7)
- added R203: DNP, Resistor_SMD:R_0402_1005Metric, F.Cu at (71.2, 101.7)
- added REF**: SMD_BD5.6-L5.6-W5.6-D3.6, LCSC_Connector:SMD_BD5.6-L5.6-W5.6-D3.6, F.Cu at (93.3, 85.9)
- added REF**: SMD_BD5.6-L5.6-W5.6-D3.6, LCSC_Connector:SMD_BD5.6-L5.6-W5.6-D3.6, F.Cu at (63.3, 52.2)
- added REF**: SMD_BD5.6-L5.6-W5.6-D3.6, LCSC_Connector:SMD_BD5.6-L5.6-W5.6-D3.6, F.Cu at (118.3, 39.1)
- added REF**: SMD_BD5.6-L5.6-W5.6-D3.6, LCSC_Connector:SMD_BD5.6-L5.6-W5.6-D3.6, F.Cu at (63.3, 85.9)
- added REF**: SMD_BD5.6-L5.6-W5.6-D3.6, LCSC_Connector:SMD_BD5.6-L5.6-W5.6-D3.6, F.Cu at (38.3, 39.1)
- added REF**: SMD_BD5.6-L5.6-W5.6-D3.6, LCSC_Connector:SMD_BD5.6-L5.6-W5.6-D3.6, F.Cu at (93.3, 52.2)
- added REF**: SMD_BD5.6-L5.6-W5.6-D3.6, LCSC_Connector:SMD_BD5.6-L5.6-W5.6-D3.6, F.Cu at (38.3, 94.1)
- added REF**: SMD_BD5.6-L5.6-W5.6-D3.6, LCSC_Connector:SMD_BD5.6-L5.6-W5.6-D3.6, F.Cu at (118.3, 94.1)
- added U101: STM32G431CBUx, Package_DFN_QFN:QFN-48-1EP_7x7mm_P0.5mm_EP5.6x5.6mm, F.Cu at (104.5, 82.5)
- added U102: AMS1117-3.3, Package_TO_SOT_SMD:SOT-223-3_TabPin2, F.Cu at (63.3, 41.3)
- added U103: LSM6DS3, Package_LGA:LGA-14_3x2.5mm_P0.5mm_LayoutBorder3x4y, F.Cu at (51.2, 92.5)
- added U104: STSPIN250, Package_DFN_QFN:TQFN-16-1EP_3x3mm_P0.5mm_EP1.6x1.6mm, F.Cu at (111.1, 39.0)
- added U105: STSPIN250, Package_DFN_QFN:TQFN-16-1EP_3x3mm_P0.5mm_EP1.6x1.6mm, F.Cu at (54.1, 38.8)
- added U201: A7105, Package_DFN_QFN:QFN-20-1EP_4x4mm_P0.5mm_EP2.5x2.5mm, F.Cu at (87.3, 93.8)
- added Y101: Crystal_GND24_DNP, Crystal:Crystal_SMD_3225-4Pin_3.2x2.5mm, F.Cu at (111.1, 89.4)
- added Y201: Crystal_GND24_DNP, Crystal:Crystal_SMD_3225-4Pin_3.2x2.5mm, F.Cu at (86.8, 99.2)
Routing:
- removed copper zone on In2.Cu, net +BATT
- removed copper zone on In2.Cu, net /RF_Transciever/REG0A
- removed copper zone on In1.Cu, net GND
- removed copper zone on In2.Cu, net VDD
Other:
- board size 100 x 65 mm -> 100 x 70 mm
- copper layers 4 -> 2

Commit message: initial commit 420
Signed-off-by: Connor Rigby <connorr@hey.com>
Parts:
- removed BT101: Battery, LCSC_Connector:PAD_01x02
- removed M101, M102: Motor_DC_ALT, LCSC_Connector:PAD_01x02
- added SW101: SW_SPDT, LCSC_Switch:SW-TH_SS-12D16L3R, F.Cu at (78.3, 39.1)
- H101, H102, H103, H104, H105, H106, H107, H108: renamed from REF**; value SMD_BD5.6-L5.6-W5.6-D3.6 -> MountingHole_Pad
- moved C123 67.3 mm to (117.5, 79.0)
- moved C124 67.3 mm to (117.5, 81.0)
- moved D101 67.3 mm to (113.9, 79.5)
- moved R116 53.0 mm to (100.3, 100.9), turned to 90 degrees
- moved R115 51.2 mm to (98.3, 100.9), turned to 90 degrees
- moved C126 50.0 mm to (100.4, 98.0), turned to 90 degrees
- moved R114 49.5 mm to (96.4, 100.9), turned to 90 degrees
- moved C125 48.1 mm to (98.4, 98.0), turned to 90 degrees
- moved R113 47.8 mm to (94.4, 100.9), turned to 90 degrees
- moved J101 45.3 mm to (104.1, 75.8)
- moved U103 44.5 mm to (95.4, 97.2), turned to 90 degrees
- moved U201 40.3 mm to (49.4, 80.3), turned to 90 degrees
- moved Y201 37.0 mm to (54.7, 80.8), turned to 90 degrees
- moved C216 36.1 mm to (47.2, 84.8), turned to 90 degrees
- moved C217 34.7 mm to (49.2, 84.8), turned to 90 degrees
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Connections:
- H101 pad 1: (no net) -> GND
- H102 pad 1: (no net) -> GND
- H103 pad 1: (no net) -> GND
- H104 pad 1: (no net) -> GND
- H105 pad 1: (no net) -> GND
- H106 pad 1: (no net) -> GND
- H107 pad 1: (no net) -> GND
- H108 pad 1: (no net) -> GND

Commit message: initial commit
Signed-off-by: Connor Rigby <connorr@hey.com>
Parts:
- added BT101: Battery, Connector_JST:JST_PH_B2B-PH-K_1x02_P2.00mm_Vertical, F.Cu at (65.1, 39.2)
- added BT102: Battery_Cell, Battery:BatteryHolder_Seiko_MS621F, F.Cu at (108.2, 75.1)
- added C129: C_0805_4u7_X5R, Capacitor_SMD:C_0805_2012Metric, F.Cu at (110.4, 89.1)
- added C130: C_0805_4u7_X5R, Capacitor_SMD:C_0805_2012Metric, F.Cu at (116.3, 85.2)
- added C131: C_0805_1u_X7R, Capacitor_SMD:C_0805_2012Metric, F.Cu at (89.8, 64.0)
- added C132: C_0805_1u_X7R, Capacitor_SMD:C_0805_2012Metric, F.Cu at (67.1, 66.0)
- added D106: BAT54C, Package_TO_SOT_SMD:SOT-23, F.Cu at (114.3, 87.2)
- added JM1: JM1, Connector_PinHeader_2.00mm:PinHeader_1x06_P2.00mm_Horizontal, F.Cu at (92.5, 59.1)
- added JM2: JM2, Connector_PinHeader_2.00mm:PinHeader_1x06_P2.00mm_Horizontal, F.Cu at (64.1, 69.1)
- added REF**: Fiducial_0.75mm_Mask1.5mm, Fiducial:Fiducial_0.75mm_Mask1.5mm, F.Cu at (124.0, 89.4)
- added REF**: Fiducial_0.75mm_Mask1.5mm, Fiducial:Fiducial_0.75mm_Mask1.5mm, F.Cu at (32.2, 89.4)
- added REF**: Fiducial_0.75mm_Mask1.5mm, Fiducial:Fiducial_0.75mm_Mask1.5mm, F.Cu at (32.4, 39.0)
- added REF**: Johanson_2450AT18x100, RF_Antenna:Johanson_2450AT18x100, F.Cu at (46.6, 89.7)
- added TP101: RESET, TestPoint:TestPoint_Pad_D1.0mm, F.Cu at (114.4, 82.9)
- added Y102: Q13FC1350000400, Crystal:Crystal_SMD_3215-2Pin_3.2x1.5mm, F.Cu at (111.8, 83.6)
- C104, C111: value C_0402_1nf_X7R -> C_0402_DNP
- C201: value C_0402_2u2_X5R -> C_805_DNP; footprint Capacitor_SMD:C_0402_1005Metric -> Capacitor_SMD:C_0805_2012Metric
- R102, R107: value 18k -> 39k
- R114: value R_0402_4k7 -> R_0402_1k
- R115: value R_0402_4k7 -> R_1206_DNP; footprint Resistor_SMD:R_0402_1005Metric -> Resistor_SMD:R_1206_3216Metric
- R116: value R_0402_1k -> R_1206_DNP; footprint Resistor_SMD:R_0402_1005Metric -> Resistor_SMD:R_1206_3216Metric
- moved R116 76.2 mm to (49.6, 44.1), turned to -90 degrees
- moved C111 71.9 mm to (109.2, 84.6), turned to 135 degrees
- moved R115 57.8 mm to (109.4, 44.1), turned to -90 degrees
- moved R114 54.9 mm to (45.5, 80.3), turned to 0 degrees
- moved R113 53.5 mm to (45.5, 79.3), turned to 0 degrees
- moved C126 51.5 mm to (51.6, 81.5), turned to 0 degrees
- moved U103 50.1 mm to (48.5, 79.5), turned to 0 degrees
- moved C125 50.0 mm to (51.6, 80.3), turned to 0 degrees
- moved C104 37.5 mm to (110.7, 86.1), turned to -45 degrees
- moved J101 33.7 mm to (77.2, 96.3), turned to 180 degrees
- moved C123 28.9 mm to (91.6, 92.0), turned to 45 degrees
- moved D101 25.7 mm to (92.3, 93.5), turned to 45 degrees
- moved R111 22.1 mm to (76.6, 45.9), turned to 0 degrees
- moved R112 21.3 mm to (79.8, 45.9), turned to 0 degrees
- moved Y201 18.6 mm to (60.6, 98.4), turned to 0 degrees
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Connections:
- net /M2_PH renamed /M2_DIR
- net /SYS_JTCK renamed /JTCK
- net /SYS_JTDI renamed /JTDI
- net /SYS_JTDO renamed /JTDO
- net /SYS_JTMS renamed /JTMS
- C101 pad 1: /MC_STBY_RESET -> /~{RESET}
- C104 pad 1: VDDA -> /OSC32_IN
- C110 pad 1: /MC_STBY_RESET -> /~{RESET}
- C111 pad 1: VDDA -> /OSC32_OUT
- C115 pad 1: VDD -> Net-(U101-VBAT)
- C124 pad 1: /~{RST} -> /~{RESET}
- J101 pad 12: /~{RST} -> /JTRST
- R101 pad 2: /MC_STBY_RESET -> /~{RESET}
- R102 pad 1: /M1_EN -> /M1_EN_FAULT
- R102 pad 2: /M1_EN_FAULT -> VDD
- R106 pad 2: /MC_STBY_RESET -> /~{RESET}
- R107 pad 1: /M2_EN -> /M2_EN_FAULT
- R107 pad 2: /M2_EN_FAULT -> VDD
- R113 pad 2: /IMU_I2C_CONFIG -> Net-(U103-SDX)
- R114 pad 2: /I2C1_SDA -> Net-(U103-SCX)
- R115 pad 1: VDD -> /M1_SENSE
- R115 pad 2: /I2C1_SCL -> GND
- R116 pad 1: VDD -> /M2_SENSE
- R116 pad 2: /IMU_CS -> GND
- SW101 pad 2: Net-(BT101-+) -> /VBAT_IN
- U101 pad 1: VDD -> Net-(U101-VBAT)
- U101 pad 10: /LPUART1_TX -> /IMU_IRQ2
- U101 pad 11: /LPUART1_RX -> /OPAMP1_WINP
- U101 pad 12: /~{SPI1_SS} -> /M2_REF
- U101 pad 13: /SPI1_SCK -> /M1_PWM
- U101 pad 14: /SPI1_MISO -> /M1_REF
- U101 pad 15: /SPI1_MOSI -> /M1_SENSE
- U101 pad 16: /RF_IRQ -> /IMU_NSS
- U101 pad 17: unconnected-(U101-PB0-Pad17) -> /M2_SENSE
- U101 pad 18: unconnected-(U101-PB1-Pad18) -> /VBATT_SENSE
- U101 pad 2: unconnected-(U101-PC13-Pad2) -> /IMU_IRQ1
- U101 pad 22: unconnected-(U101-PB10-Pad22) -> /LPUART1_RX
- U101 pad 24: /M2_EN -> /LPUART1_TX
- U101 pad 25: /MC_STBY_RESET -> /RADIO_NSS
- U101 pad 26: /M1_SENSE -> /SPI2_SCK
- U101 pad 27: /M2_SENSE -> /SPI2_MISO
- U101 pad 28: /M2_EN_FAULT -> /SPI2_MOSI
- U101 pad 29: /M1_EN_FAULT -> /M2_ENC_P
- U101 pad 3: unconnected-(U101-PC14-Pad3) -> /OSC32_IN
- U101 pad 30: /M1_PWM -> /M1_ENC_P
- U101 pad 31: /M2_PWM -> /M1_ENC_N
- U101 pad 32: /M1_EN -> /M1_DIR
- U101 pad 33: /M1_PH -> /VBAT_STATUS
- U101 pad 39: unconnected-(U101-PC10-Pad39) -> /SPI3_SCK
- U101 pad 4: unconnected-(U101-PC15-Pad4) -> /OSC32_OUT
- U101 pad 40: unconnected-(U101-PC11-Pad40) -> /SPI3_MISO
- U101 pad 42: unconnected-(U101-PB4-Pad42) -> /JTRST
- U101 pad 43: /IMU_INT1 -> /SPI3_MOSI
- U101 pad 44: /IMU_INT2 -> /M1_EN_FAULT
- U101 pad 45: /I2C1_SDA -> /M2_EN_FAULT
- U101 pad 46: /I2C1_SCL -> /M2_ENC_N
- U101 pad 7: /~{RST} -> /~{RESET}
- U101 pad 8: /VBATT_SENSE -> /RADIO_IRQ
- U101 pad 9: unconnected-(U101-PA1-Pad9) -> /M2_PWM
- U103 pad 1: /IMU_I2C_CONFIG -> /SPI3_MISO
- U103 pad 12: /IMU_CS -> /IMU_NSS
- U103 pad 13: /I2C1_SCL -> /SPI3_SCK
- U103 pad 14: /I2C1_SDA -> /SPI3_MOSI
- U103 pad 2: /IMU_I2C_CONFIG -> Net-(U103-SDX)
- U103 pad 3: /IMU_I2C_CONFIG -> Net-(U103-SCX)
- U103 pad 4: /IMU_INT1 -> /IMU_IRQ1
- U103 pad 9: /IMU_INT2 -> /IMU_IRQ2
- U104 pad 1: /M1_PH -> /M1_DIR
- U104 pad 11: VDDA -> /M1_REF
- U104 pad 14: /MC_STBY_RESET -> /~{RESET}
- U105 pad 11: VDDA -> /M2_REF
- U105 pad 14: /MC_STBY_RESET -> /~{RESET}
- U201 pad 11: /~{SPI1_SS} -> /RADIO_NSS
- U201 pad 12: /SPI1_SCK -> /SPI2_SCK
- U201 pad 14: /SPI1_MOSI -> /SPI2_MOSI
- U201 pad 16: /SPI1_MISO -> /SPI2_MISO
- U201 pad 17: /RF_IRQ -> /RADIO_IRQ
Routing:
- net /~{RESET}: track 0.00 -> 173.0 mm, vias 0 -> 2
- net /M2_EN_FAULT: track 0.00 -> 124.0 mm, vias 0 -> 2
- net /M1_EN_FAULT: track 0.00 -> 123.3 mm, vias 0 -> 2
- net /M2_DIR: track 0.00 -> 109.1 mm, vias 0 -> 2
- net /IMU_IRQ1: track 0.00 -> 105.3 mm, vias 0 -> 4
- net /M2_PWM: track 0.00 -> 99.0 mm, vias 0 -> 2
- net GND: track 0.00 -> 94.8 mm, vias 0 -> 78
- net /M1_DIR: track 0.00 -> 93.2 mm, vias 0 -> 2
- net /M1_REF: track 0.00 -> 93.1 mm, vias 0 -> 2
- net /M1_SENSE: track 0.00 -> 92.2 mm, vias 0 -> 6
- net /M2_SENSE: track 0.00 -> 92.0 mm, vias 0 -> 6
- net /SPI3_MOSI: track 0.00 -> 92.0 mm, vias 0 -> 4
- net /M2_REF: track 0.00 -> 90.4 mm, vias 0 -> 2
- net /M2_ENC_N: track 0.00 -> 90.1 mm, vias 0 -> 2
- net /SPI3_MISO: track 0.00 -> 88.2 mm, vias 0 -> 4
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- added copper zone on F.Cu, net +BATT
- added copper zone on In2.Cu, net +BATT
- added copper zone on B.Cu, net /M1_OUTA1
- added copper zone on F.Cu, net /M1_OUTA1
- added copper zone on B.Cu, net /M1_OUTA2
- added copper zone on F.Cu, net /M1_OUTA2
- added copper zone on B.Cu, net /M1_SENSE
- added copper zone on F.Cu, net /M1_SENSE
- added copper zone on B.Cu, net /M2_OUTA1
- added copper zone on F.Cu, net /M2_OUTA1
- added copper zone on B.Cu, net /M2_OUTA2
- added copper zone on F.Cu, net /M2_OUTA2
- added copper zone on B.Cu, net /M2_SENSE
- added copper zone on F.Cu, net /M2_SENSE
- added copper zone on F.Cu, net /VBAT_IN
- added copper zone on B.Cu, net GND
- added copper zone on F.Cu, net GND
- added copper zone on In1.Cu, net GND
- added copper zone on B.Cu, net VDD
- added copper zone on F.Cu, net VDD
- added copper zone on In2.Cu, net VDD
Other:
- outline, holes or cut-outs redrawn
- copper layers 2 -> 4
