File: hardware/150g-battlebot-pcb.kicad_sch (KiCad schematic)
At the start: 16 parts, among them U101 STM32G431C6Ux, U102 MIC5504-3.3YM5

Commit message: pcb initialize
Signed-off-by: Connor Rigby <connorr@hey.com>
Parts:
- removed BT101: Battery, symbol Device:Battery
- removed BT102: Battery_Cell, symbol Device:Battery_Cell
- removed C101, C102: C_0805_1u_X7R, Capacitor_SMD:C_0805_2012Metric, symbol LCSC_Capacitor:C_0805_1u_X7R
- removed C103, C105, C106, C107, C108, C110: C_0402_100nf_X7R, Capacitor_SMD:C_0402_1005Metric, symbol LCSC_Capacitor:C_0402_100nf_X7R
- removed C104: C_0805_4u7_X5R, Capacitor_SMD:C_0805_2012Metric, symbol LCSC_Capacitor:C_0805_4u7_X5R
- removed C109: C_0402_1u_X5R, Capacitor_SMD:C_0402_1005Metric, symbol LCSC_Capacitor:C_0402_1u_X5R
- removed D101: BAT54C, Package_TO_SOT_SMD:SOT-23, symbol Diode:BAT54C
- removed FB101: FerriteBead_Small, symbol Device:FerriteBead_Small
- removed U101: STM32G431C6Ux, Package_DFN_QFN:QFN-48-1EP_7x7mm_P0.5mm_EP5.6x5.6mm, symbol MCU_ST_STM32G4:STM32G431C6Ux
- removed U102: MIC5504-3.3YM5, Package_TO_SOT_SMD:SOT-23-5, symbol Regulator_Linear:MIC5504-3.3YM5
Other:
- added sheet Application (Application.kicad_sch)
- added sheet MotorDrivers (MotorDrivers.kicad_sch)
- added sheet PowerInput (PowerInput.kicad_sch)
- added sheet RF (RF.kicad_sch)
- added sheet Sensors (Sensors.kicad_sch)

Commit message: asdf
Signed-off-by: Connor Rigby <connorr@hey.com>
Changed lines of the file:
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@@
 (kicad_sch (version 20230121) (generator eeschema)
   (paper "A4")
-  (sheet (at 96.52 127) (size 30.48 22.86) (fields_autoplaced)
-    (stroke (width 0.1524) (type solid))
-    (fill (color 0 0 0 0.0000))
-    (property "Sheetname" "RF" (at 96.52 126.2884 0)
-      (effects (font (size 1.27 1.27)) (justify left bottom))
-    )
-    (property "Sheetfile" "RF.kicad_sch" (at 96.52 150.4446 0)
-      (effects (font (size 1.27 1.27)) (justify left top))
-    )
-    (instances
-      (project "150g-battlebot-pcb"
-        (path "/80268558-ae7f-45c2-9b9a-7f2ee458c642" (page "6"))
-      )
-    )
-  )
   (sheet (at 231.14 29.21) (size 16.51 15.24) (fields_autoplaced)
     (stroke (width 0.1524) (type solid))
@@
     (instances
       (project "150g-battlebot-pcb"
+        (path "/80268558-ae7f-45c2-9b9a-7f2ee458c642" (page "5"))
+      )
+    )
+  )
+  (sheet (at 82.55 121.92) (size 25.4 33.02) (fields_autoplaced)
+    (stroke (width 0.1524) (type solid))
+    (fill (color 0 0 0 0.0000))
+    (property "Sheetname" "RF" (at 82.55 121.2084 0)
+      (effects (font (size 1.27 1.27)) (justify left bottom))
+    )
+    (property "Sheetfile" "RF.kicad_sch" (at 82.55 155.5246 0)
+      (effects (font (size 1.27 1.27)) (justify left top))
+    )
+    (instances
+      (project "150g-battlebot-pcb"
         (path "/80268558-ae7f-45c2-9b9a-7f2ee458c642" (page "2"))
       )
     )
   )
-  (sheet (at 144.78 52.07) (size 29.21 20.32) (fields_autoplaced)
+  (sheet (at 25.4 24.13) (size 29.21 20.32) (fields_autoplaced)
     (stroke (width 0.1524) (type solid))
     (fill (color 0 0 0 0.0000))
-    (property "Sheetname" "PowerInput" (at 144.78 51.3584 0)
+    (property "Sheetname" "PowerInput" (at 25.4 23.4184 0)
       (effects (font (size 1.27 1.27)) (justify left bottom))
     )
-    (property "Sheetfile" "PowerInput.kicad_sch" (at 144.78 72.9746 0)
+    (property "Sheetfile" "PowerInput.kicad_sch" (at 25.4 45.0346 0)
       (effects (font (size 1.27 1.27)) (justify left top))
     )

Commit message: asdf
Signed-off-by: Connor Rigby <connorr@hey.com>
Other:
- sheet Application ports: added BAT_SENSE, FAULT, IMU_INT1, IMU_INT2, M1_DIR, M1_ENCA, M1_ENCB, M1_PWM, M2_DIR, M2_ENCA, M2_ENCB, M2_PWM, M3_DIR, M3_ENCA, M3_ENCB, M3_PWM, M4_DIR, M4_ENCA, M4_ENCB, M4_PWM, REF, RF_GIO2, SPI1_MISO, SPI1_MOSI, SPI1_SCK, ~{IMU_CS}, ~{RESET}, ~{RF_CS}; removed none
- sheet MotorDrivers ports: added EN_FAULT, M1_ENCA, M1_ENCB, M1_PH, M1_PWM, M2_ENCA, M2_ENCB, M2_PH, M2_PWM, M3_ENCA, M3_ENCB, M3_PH, M3_PWM, M4_ENCA, M4_ENCB, M4_PH, M4_PWM, REF, ~{RESET}; removed none
- sheet RF ports: added GIO1, GIO2, SCK, SCS, SDIO; removed none
- sheet Sensors ports: added INT1, INT2, MISO, MOSI, SCLK, VBAT_SENSE, ~{CS}; removed none
- note added: "Battery +VS"
- note added: "VDD"
