File: hardware/PowerInput.kicad_sch (KiCad schematic)
At the start: 6 parts, among them U102 MIC5504-3.3YM5

Commit message: asdf
Signed-off-by: Connor Rigby <connorr@hey.com>
Parts:
- added C303: C_0805_4u7_X5R, Capacitor_SMD:C_0805_2012Metric, symbol LCSC_Capacitor:C_0805_4u7_X5R
- added C304: C_0402_1u_X5R, Capacitor_SMD:C_0402_1005Metric, symbol LCSC_Capacitor:C_0402_1u_X5R
- added FB301: FerriteBead_Small, Inductor_SMD:L_0402_1005Metric, symbol Device:FerriteBead_Small
- added SW101: SW_SPDT, LCSC_Switch:SW-TH_SS-12D16L3R, symbol Switch:SW_SPDT
- BT102: footprint (none) -> Battery:BatteryHolder_Seiko_MS621F
Connections:
- net GND: now also C303.2, C304.2
- net VDD: now reaches C102.1, U102.5 (VOUT)
- net VDD: now also D101.2
- net VIN: now reaches C101.1, U102.1 (VIN), U102.3 (EN)
- net VIN: now also SW101.3 (C); no longer BT101.1 (+), D101.2
- net +BATT: now reaches BT102.1 (+), D101.1
- net at D101.3: now also C303.1, FB301.1
- new net VDDA: C304.1, FB301.2
- new net VS: BT101.1 (+), SW101.2 (B)
Other:
- moved on the sheet: BT101, BT102, D101

Commit message: asdf
Signed-off-by: Connor Rigby <connorr@hey.com>
Connections:
- net +BATT: now also C303.1, D101.3; no longer BT102.1 (+), D101.1
- net VDD: now also FB301.1
- new net: BT102.1 (+), D101.1
Other:
- moved on the sheet: C303, C304, FB301
