File: hardware/RF.kicad_sch (KiCad schematic)
At the start: 0 parts

Commit message: asdf
Signed-off-by: Connor Rigby <connorr@hey.com>
Parts:
- added AE201: Antenna_Chip, symbol Device:Antenna_Chip
- added C201: C_805_DNP, Capacitor_SMD:C_0805_2012Metric, symbol LCSC_Capacitor:C_805_DNP
- added C202, C204: C_0402_2u2_X5R, Capacitor_SMD:C_0402_1005Metric, symbol LCSC_Capacitor:C_0402_2u2_X5R
- added C203, C206, C207, C208, C209, C211, C214, C215, C216, C217, C218, C219, C220: C_0402_DNP, Capacitor_SMD:C_0402_1005Metric, symbol LCSC_Capacitor:C_0402_DNP
- added C205: C_0402_100nf_X7R, Capacitor_SMD:C_0402_1005Metric, symbol LCSC_Capacitor:C_0402_100nf_X7R
- added C210: C_0402_22p_C0G, Capacitor_SMD:C_0402_1005Metric, symbol LCSC_Capacitor:C_0402_22p_C0G
- added C212: C_0402_100p_C0G, Capacitor_SMD:C_0402_1005Metric, symbol LCSC_Capacitor:C_0402_100p_C0G
- added C213: C_0402_10n_C0G, Capacitor_SMD:C_0402_1005Metric, symbol LCSC_Capacitor:C_0402_10n_C0G
- added L202, L203, L204: L_0402_DNP, Inductor_SMD:L_0402_1005Metric, symbol LCSC_Inductor:L_0402_DNP
- added R201, R203: DNP, Resistor_SMD:R_0402_1005Metric, symbol LCSC_Resistor:R_0402_DNP
- added R202: 200, Resistor_SMD:R_0402_1005Metric, symbol LCSC_Resistor:R_0402_DNP
- added U103: A7105, Package_DFN_QFN:QFN-20-1EP_4x4mm_P0.5mm_EP2.5x2.5mm, symbol LCSC_RF_Transciever_ICs:A7105
- added Y201: 16_mhz, Crystal:Crystal_SMD_3225-4Pin_3.2x2.5mm, symbol LCSC_Crystal:Crystal_GND24_DNP
Connections:
- new net: C209.2, R202.2, U103.6 (VT)
- new net: C215.1, U103.8 (XI), Y201.1
- new net: C214.1, U103.9 (XO), Y201.3
- new net: C206.2, C210.1, C216.1, L202.2, L204.2
- new net: C213.2, R202.1
- new net: AE201.1 (FEED), C219.2, R203.2
- new net ANT: C217.1, C218.1, C220.2, L204.1, R203.1
- new net BPBG: C208.2, U103.2 (BPBG)
- new net GIO1: U103.16 (GIO1)
- new net GIO2: U103.17 (GIO2)
- new net GND: AE201.2 (PCB_Trace), C201.2, C202.2, C203.1, C204.2, C205.2, C207.1, C208.1, C209.1, C211.1, C212.2, C213.1, C214.2, C215.2, C216.2, C217.2, C218.2, C219.1, C220.1, L202.1, U103.15 (GND), U103.21 (EP), U103.7 (GND), Y201.2, Y201.4
- new net REG0A: C201.1, C205.1, C211.2, C212.1, L203.2, R201.1, U103.10 (VDA3), U103.20 (VDA1)
- new net RFI: C210.2, U103.3 (RFI)
- new net RFO: C206.1, L203.1, U103.4 (RFO)
- new net RSSI: C207.2, U103.1 (RSSI)
- new net SCK: U103.12 (SCK)
- new net SCS: U103.11 (SCS)
- new net SDIO: U103.14 (SDIO)
- new net VDA2: C203.2, R201.2, U103.5 (VDA2)
- new net VDD: C202.1, C204.1, U103.13 (DVDD), U103.19 (REGI)
- no-connect marks 0 -> 1

Commit message: asdf
Signed-off-by: Connor Rigby <connorr@hey.com>
Parts:
- AE201: footprint (none) -> LCSC_Antenna:IPEX-SMD_BWIPX-1-001E
Changed lines of the file:
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@@
       (effects (font (size 1.27 1.27)) (justify right))
     )
-    (property "Footprint" "" (at 38.1 31.115 0)
+    (property "Footprint" "LCSC_Antenna:IPEX-SMD_BWIPX-1-001E" (at 38.1 31.115 0)
       (effects (font (size 1.27 1.27)) hide)
     )
