File: hardware/Sensors.kicad_sch (KiCad schematic)
At the start: 1 part, among them U107 LIS3DH

Commit message: asdf
Signed-off-by: Connor Rigby <connorr@hey.com>
Parts:
- added C501, C502: C_0402_100nf_X7R, Capacitor_SMD:C_0402_1005Metric, symbol LCSC_Capacitor:C_0402_100nf_X7R
- added R501, R502: R_0603_DNP, Resistor_SMD:R_0603_1608Metric, symbol LCSC_Resistor:R_0603_DNP
Connections:
- net at U107.1 (VDD_IO): now also U107.14 (VDD), C501.1, C502.1
- net GND: now reaches U107.10 (GND), U107.12 (GND), U107.5 (GND)
- net GND: now also U107.13 (ADC3), U107.15 (ADC2), U107.16 (ADC1), C501.2, C502.2, R501.2
- net INT1: now reaches U107.11 (INT1)
- net SCLK: now reaches U107.4 (SCL/SPC)
- net MOSI: now reaches U107.6 (SDA/SDI/SDO)
- net MISO: now reaches U107.7 (SDO/SA0)
- net ~{CS}: now reaches U107.8 (CS)
- net INT2: now reaches U107.9 (INT2)
- new net VBAT_SENSE: R501.1, R502.2
- new net VS: R502.1
Other:
- moved on the sheet: U107

Commit message: asdf
Signed-off-by: Connor Rigby <connorr@hey.com>
Parts:
- removed C501: C_0402_100nf_X7R, Capacitor_SMD:C_0402_1005Metric, symbol LCSC_Capacitor:C_0402_100nf_X7R
- added C501: C_0402_DNP, Capacitor_SMD:C_0402_1005Metric, symbol LCSC_Capacitor:C_0402_DNP
Connections:
- net GND: now also C501.2
- net VDD: now reaches C502.1, U107.1 (VDD_IO), U107.14 (VDD)
- net VDD: now also C501.1
Changed lines of the file:
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@@
   (junction (at 76.2 55.88) (diameter 0) (color 0 0 0 0)
+  )
+  (junction (at 38.1 25.4) (diameter 0) (color 0 0 0 0)
   )
   (junction (at 54.61 25.4) (diameter 0) (color 0 0 0 0)
@@
     )
   )
+  (symbol (lib_id "power:VDD") (at 38.1 25.4 0) (unit 1)
+    (in_bom yes) (on_board yes) (dnp no) (fields_autoplaced)
+    (property "Reference" "#PWR0507" (at 38.1 29.21 0)
+      (effects (font (size 1.27 1.27)) hide)
+    )
+    (property "Value" "VDD" (at 38.1 20.32 0)
+      (effects (font (size 1.27 1.27)))
+    )
+    (property "Footprint" "" (at 38.1 25.4 0)
+      (effects (font (size 1.27 1.27)) hide)
+    )
+    (property "Datasheet" "" (at 38.1 25.4 0)
+      (effects (font (size 1.27 1.27)) hide)
+    )
+    (pin "1")
+    (instances
+      (project "150g-battlebot-pcb"
+        (path "/80268558-ae7f-45c2-9b9a-7f2ee458c642/f96a4b82-6d44-4b23-8cfe-3bbd7486daa6"
+          (reference "#PWR0507") (unit 1)
+        )
+      )
+    )
+  )
   (symbol (lib_id "power:GND") (at 50.8 30.48 0) (unit 1)
     (in_bom yes) (on_board yes) (dnp no) (fields_autoplaced)
@@
         (path "/80268558-ae7f-45c2-9b9a-7f2ee458c642/f96a4b82-6d44-4b23-8cfe-3bbd7486daa6"
           (reference "#PWR0504") (unit 1)
-        )
-      )
-    )
-  )
-  (symbol (lib_id "LCSC_Capacitor:C_0402_100nf_X7R") (at 38.1 27.94 0) (unit 1)
-    (in_bom no) (on_board yes) (dnp no)
-    (property "Reference" "C501" (at 30.48 26.67 0)
-      (effects (font (size 1.27 1.27)) (justify left))
-    )
-    (property "Value" "C_0402_100nf_X7R" (at 38.354 29.972 0)
-      (effects (font (size 1.27 1.27)) (justify left) hide)
-    )
-    (property "Footprint" "Capacitor_SMD:C_0402_1005Metric" (at 38.1 27.94 0)
-      (effects (font (size 1.27 1.27)) hide)
-    )
-    (property "Datasheet" "https://datasheet.lcsc.com/lcsc/1811141731_FH--Guangdong-Fenghua-Advanced-Tech-0402B104K500NT_C110251.pdf" (at 38.1 27.94 0)
-      (effects (font (size 1.27 1.27)) hide)
-    )
-    (property "MPN" "0402B104K500NT" (at 38.1 27.94 0)
-      (effects (font (size 1.27 1.27)) hide)
-    )
-    (property "LCSC" "C110251" (at 38.1 27.94 0)
-      (effects (font (size 1.27 1.27)) hide)
-    )
-    (property "Capacitance" "100nf" (at 30.48 29.21 0)
-      (effects (font (size 1.27 1.27)) (justify left))
-    )
-    (property "Voltage" "50V" (at 38.1 27.94 0)
-      (effects (font (size 1.27 1.27)) hide)
-    )
-    (property "Temperature" "X7R" (at 38.1 27.94 0)
-      (effects (font (size 1.27 1.27)) hide)
-    )
-    (pin "1")
-    (pin "2")
-    (instances
-      (project "150g-battlebot-pcb"
-        (path "/80268558-ae7f-45c2-9b9a-7f2ee458c642/f96a4b82-6d44-4b23-8cfe-3bbd7486daa6"
-          (reference "C501") (unit 1)
         )
       )
@@
         )
       )
+    )
+  )
+  (symbol (lib_id "LCSC_Capacitor:C_0402_DNP") (at 38.1 27.94 0) (unit 1)
+    (in_bom no) (on_board yes) (dnp no) (fields_autoplaced)
+    (property "Reference" "C501" (at 35.56 26.6763 0)
+      (effects (font (size 1.27 1.27)) (justify right))
+    )
+    (property "Value" "C_0402_DNP" (at 38.354 29.972 0)
+      (effects (font (size 1.27 1.27)) (justify left) hide)
+    )
+    (property "Footprint" "Capacitor_SMD:C_0402_1005Metric" (at 38.1 27.94 0)
+      (effects (font (size 1.27 1.27)) hide)
+    )
+    (property "Datasheet" "~" (at 38.1 27.94 0)
+      (effects (font (size 1.27 1.27)) hide)
+    )
+    (property "Capacitance" "10uF" (at 35.56 29.2163 0)
+      (effects (font (size 1.27 1.27)) (justify right))
+    )
+    (pin "1")
+    (pin "2")
+    (instances
+      (project "150g-battlebot-pcb"
+        (path "/80268558-ae7f-45c2-9b9a-7f2ee458c642/f96a4b82-6d44-4b23-8cfe-3bbd7486daa6"
+          (reference "C501") (unit 1)
+        )
+      )
